File: orphkicad.kicad_sch (KiCad schematic)
At the start: 41 parts, among them J1 USB_C_Receptacle_USB2.0_16P, J2 SWD, SW1 BTN_BOOT, SW2 BTN_RST, SW3 BTN_USR, U1 RP2040, U2 W25Q16JVUXIQ, U3 USBLC6-2SC6, U5 XC6206PxxxMR, X1 X322512MOB4SI 12pF

Commit message: Change LCSC id, move trace, add gnd via
Parts:
- X1: LCSC C9002 -> C70565
Changed lines of the file:
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@@
 			)
 		)
-		(property "LCSC" "C9002"
+		(property "LCSC" "C70565"
 			(at 241.3 39.37 0)
 			(effects
